File: rainbow2-rp2040/rainbow2-rp2040.kicad_pcb (KiCad board)
At the start: 2 copper layers, 45 x 99.5 mm, 24 parts, among them J1 SCR_SENSE, J10 E1, J11 E2, J2 2ND_PWR, J3 BT1, J4 BT2, J5 BT3, J6 BT4, J7 BT5, J8 BT6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

Commit message: update iidx_pcb_rev2
Parts:
- removed R3, R4: 10k, Resistor_THT:R_Axial_DIN0207_L6.3mm_D2.5mm_P10.16mm_Horizontal
- removed RN1: 10K, Resistor_THT:R_Array_SIP9
- R1, R2: value 10k -> ???
- U2, U3: footprint Package_SO:SOP-16_3.9x9.9mm_P1.27mm -> Package_DIP:DIP-16_W7.62mm_Socket
- moved R1 15.6 mm to (103.0, 64.5)
- moved J10 12.5 mm to (108.5, 75.0)
- moved J11 12.5 mm to (108.5, 82.5)
- moved J3 12.5 mm to (108.5, 90.0)
- moved J4 12.5 mm to (108.5, 97.5)
- moved J5 12.5 mm to (108.5, 105.0)
- moved J6 12.5 mm to (108.5, 112.5)
- moved J7 12.5 mm to (108.5, 120.0)
- moved J8 12.5 mm to (108.5, 127.5)
- moved J9 12.5 mm to (108.5, 135.0)
- moved U3 9.56 mm to (120.0, 86.0)
- moved U2 7.13 mm to (120.0, 111.5)
- moved R2 6.67 mm to (103.0, 69.0)
- moved REF** 1.79 mm to (132.7, 87.0)
Connections:
- R1 pad 1: HE1 -> K1
- R1 pad 2: GND -> +3V3
- R2 pad 1: HE2 -> K2
- R2 pad 2: GND -> +3V3
- U1 pad 12: LK2 -> K2
- U1 pad 13: LK1 -> K1
- U1 pad 21: unconnected-(U1-3V3-Pad21) -> +3V3
- U3 pad 12: LK2 -> unconnected-(U3-O5-Pad12)
- U3 pad 13: LK1 -> unconnected-(U3-O4-Pad13)
- U3 pad 4: K1 -> unconnected-(U3-I4-Pad4)
- U3 pad 5: K2 -> unconnected-(U3-I5-Pad5)
Routing:
- net HBT7: track 43.4 -> 16.2 mm
- net HBT6: track 37.6 -> 11.3 mm
- net LBT7: track 59.4 -> 81.2 mm, vias 2 -> 1
- net +5V: track 135.8 -> 114.3 mm
- net HBT5: track 31.8 -> 10.9 mm
- net LBT6: track 55.1 -> 75.1 mm, vias 2 -> 1
- net LK2: track 19.9 -> 0.00 mm, vias 2 -> 0
- net LK1: track 18.5 -> 0.00 mm, vias 2 -> 0
- net LBT5: track 50.5 -> 68.8 mm, vias 2 -> 1
- net +3V3: track 0.00 -> 17.3 mm, vias 0 -> 1
- net LBT4: track 45.8 -> 62.5 mm, vias 2 -> 1
- net HBT1: track 14.5 -> 29.6 mm
- net LBT3: track 41.5 -> 56.4 mm, vias 2 -> 1
- net HE2: track 41.2 -> 26.7 mm
- net LBT2: track 37.2 -> 50.4 mm, vias 2 -> 1
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Other:
- outline, holes or cut-outs redrawn
- board text added: "RBC:J:B:A:2024090X00"
- board text removed: "RBC:J:B:A:2024081800"
