File: rainbow2-rp2040/rainbow2-rp2040.kicad_sch (KiCad schematic)
At the start: 23 parts, among them J1 SCR_SENSE, J10 E1, J11 E2, J2 2ND_PWR, J3 BT1, J4 BT2, J5 BT3, J6 BT4, J7 BT5, J8 BT6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

Commit message: update iidx_pcb_rev2
Parts:
- removed R3, R4: 10k, Resistor_THT:R_Axial_DIN0207_L6.3mm_D2.5mm_P10.16mm_Horizontal, symbol Device:R
- removed RN1: 10K, Resistor_THT:R_Array_SIP9, symbol Device:R_Network08
- R1, R2: value 10k -> ???
- U2, U3: footprint Package_SO:SOP-16_3.9x9.9mm_P1.27mm -> Package_DIP:DIP-16_W7.62mm_Socket
Connections:
- net GND: no longer R1.2, R2.2
- net HE1: no longer R1.1
- net HE2: no longer R2.1
- net K1: now also R1.1, U1.13 (12); no longer U3.4 (I4)
- net K2: now also R2.1, U1.12 (11); no longer U3.5 (I5)
- net +3V3: now reaches U1.21 (3V3)
- net +3V3: now also R1.2, R2.2
- net LK1: no longer names the net of U3.13 (O4)
- net LK1: no longer U1.13 (12)
- net LK2: no longer names the net of U3.12 (O5)
- net LK2: no longer U1.12 (11)
- no-connect marks 19 -> 21
