File: iidx_pcb_rev2/iidx_pcb.kicad_pcb (KiCad board)
At the start: 2 copper layers, 68.6 x 52.7 mm, 11 parts, among them J101 TT, J102 BT, U101 rp2040-zero

Commit message: 溜めすぎ　人間性0点
Parts:
- added J3: PSX, Connector_PinSocket_2.54mm:PinSocket_1x07_P2.54mm_Vertical, F.Cu at (110.5, 100.3)
- added JP1: PSX3V3, Connector_PinHeader_2.54mm:PinHeader_1x02_P2.54mm_Vertical, F.Cu at (106.0, 115.6)
- added R1: 1k, Resistor_THT:R_Axial_DIN0204_L3.6mm_D1.6mm_P5.08mm_Horizontal, F.Cu at (55.9, 116.8)
- added R10: 330, Resistor_SMD:R_0805_2012Metric_Pad1.20x1.40mm_HandSolder, B.Cu at (55.2, 104.8)
- added R11: 330, Resistor_SMD:R_0805_2012Metric_Pad1.20x1.40mm_HandSolder, B.Cu at (59.1, 104.8)
- added R2: 1k, Resistor_THT:R_Axial_DIN0204_L3.6mm_D1.6mm_P5.08mm_Horizontal, F.Cu at (55.9, 119.4)
- added R3: 1k, Resistor_THT:R_Axial_DIN0204_L3.6mm_D1.6mm_P5.08mm_Horizontal, F.Cu at (55.9, 121.9)
- added R4: 1k, Resistor_THT:R_Axial_DIN0204_L3.6mm_D1.6mm_P5.08mm_Horizontal, F.Cu at (55.9, 124.5)
- added R5: 1k, Resistor_THT:R_Axial_DIN0204_L3.6mm_D1.6mm_P5.08mm_Horizontal, F.Cu at (55.9, 127.0)
- added R6: 1k, Resistor_THT:R_Axial_DIN0204_L3.6mm_D1.6mm_P5.08mm_Horizontal, F.Cu at (55.9, 129.5)
- added R7: 1k, Resistor_THT:R_Axial_DIN0204_L3.6mm_D1.6mm_P5.08mm_Horizontal, F.Cu at (55.9, 137.2)
- R8: renamed from R101; footprint Resistor_SMD:R_0805_2012Metric_Pad1.20x1.40mm_HandSolder -> Resistor_THT:R_Axial_DIN0204_L3.6mm_D1.6mm_P5.08mm_Horizontal
- R9: renamed from R102; footprint Resistor_SMD:R_0805_2012Metric_Pad1.20x1.40mm_HandSolder -> Resistor_THT:R_Axial_DIN0204_L3.6mm_D1.6mm_P5.08mm_Horizontal
- moved S2 36.8 mm to (92.1, 100.3)
- moved S1 36.3 mm to (78.7, 101.0)
- moved S3 30.6 mm to (67.9, 101.0)
- moved J2 0.70 mm to (50.8, 117.0)
- moved S4 0.64 mm to (86.4, 146.7)
- moved J1 0.44 mm to (50.8, 102.7)
- moved R8 0.40 mm to (55.2, 102.2)
- moved R9 0.40 mm to (59.1, 102.2)
- renumbered H101 to H1, H102 to H2, J101 to J1, J102 to J2, S101 to S1, S102 to S2, S103 to S3, S104 to S4, U101 to U1
Connections:
- U1 pad 15: SCR_UP -> unconnected-(U1-14-Pad15)
- U1 pad 16: SCR_DOWN -> PSX_ATT
- U1 pad 17: unconnected-(U101-26-Pad17) -> PSX_SCK
- U1 pad 18: unconnected-(U101-27-Pad18) -> PSX_CMD
- U1 pad 19: unconnected-(U101-28-Pad19) -> PSX_DAT
- U1 pad 20: unconnected-(U101-29-Pad20) -> PSX_ACK
Routing:
- net +3V3: track 69.4 -> 112.4 mm
- net PSX_ATT: track 0.00 -> 36.5 mm
- net PSX_SCK: track 0.00 -> 31.4 mm
- net Net-(J3-Pin_1): track 0.00 -> 30.8 mm
- net PSX_CMD: track 0.00 -> 26.3 mm
- net PSX_DAT: track 0.00 -> 21.2 mm
- net PSX_ACK: track 0.00 -> 16.1 mm
- net KEY_2: track 74.6 -> 66.3 mm
- net KEY_7: track 59.4 -> 66.0 mm
- net KEY_SEL: track 70.8 -> 64.9 mm
- net KEY_6: track 57.0 -> 61.9 mm
- net KEY_STA: track 67.1 -> 63.4 mm
- net KEY_3: track 54.9 -> 58.3 mm
- net SCR_LEDB: track 14.6 -> 11.9 mm, vias 1 -> 0
- net SCR_TRCB: track 76.6 -> 79.0 mm
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Other:
- board size 68.6 x 52.7 mm -> 68.6 x 55.9 mm
- board text added: "GP15(ATT)"
- board text added: "GP26(SCK)"
- board text added: "GP27(CMD)"
- board text added: "GP28(DAT)"
- board text added: "GP29(ACK)"
- board text added: "KOC:J:A:A:2025093000"
- board text added: "OPEN SOURCE, OPEN BEAT, OPEN FUTURE."
- board text removed: "KOC:J:A:A:2025021000"
