File: iidx_pcb_rev2/iidx_pcb.kicad_sch (KiCad schematic)
At the start: 5 parts, among them J2 Conn_01x05, J3 Conn_01x12, U1 RP2040-Zero

Commit message: update iidx_pcb_rev2
Parts:
- removed U1: RP2040-Zero, rp2040:RP2040-Zero, symbol rp2040-zero:RP2040-Zero
- added S1: OSHW_Logo, Symbol:OSHW-Logo2_9.8x8mm_SilkScreen, symbol Mechanical:MountingHole
- added S2: KiCad_Logo, Symbol:KiCad-Logo2_6mm_SilkScreen, symbol Mechanical:MountingHole
- added U2: rp2040-zero, mcu:rp2040-zero-tht, symbol mcu:rp2040-zero
- R1, R2: footprint Resistor_THT:R_Axial_DIN0207_L6.3mm_D2.5mm_P10.16mm_Horizontal -> Resistor_SMD:R_0805_2012Metric_Pad1.20x1.40mm_HandSolder
Connections:
- net 3V3: now also U2.21 (3V3)
- net 5V: now also U2.23 (5V)
- net GND: now also U2.22 (GND)
- net KEY_1: now also U2.6 (5)
- net KEY_2: now also U2.3 (2)
- net KEY_3: now also U2.9 (8)
- net KEY_4: now also U2.8 (7)
- net KEY_5: now also U2.7 (6)
- net KEY_6: now also U2.10 (9)
- net KEY_7: now also U2.11 (10)
- net KEY_SEL: now also U2.4 (3)
- net KEY_STA: now also U2.5 (4)
- net SCR_DOWN: now also U2.16 (15)
- net SCR_TRCA: now also U2.13 (12)
- net SCR_TRCB: now also U2.12 (11)
- net SCR_UP: now also U2.15 (14)
- no-connect marks 10 -> 9

Commit message: update footprints for rev2
Parts:
- added H101, H102: Screw, MountingHole:MountingHole_3.2mm_M3_DIN965_Pad, symbol Mechanical:MountingHole_Pad
- added S103: Librebeat, Symbol_k:Project_Librebeat_Logo, symbol Mechanical:MountingHole
- added S104: Kemono, Symbol_k:Kemono_Symbol, symbol Mechanical:MountingHole
- J101: renamed from J2; value Conn_01x05 -> TT
- J102: renamed from J3; value Conn_01x12 -> BT
- renumbered R1 to R101, R2 to R102, S1 to S101, S2 to S102, U2 to U101
Connections:
- net GND: now also H101.1, H102.1
- net 3V3 renamed +3V3
- net 5V renamed +5V
