File: iidx_pcb_rev2/iidx_pcb.kicad_sch (KiCad schematic)
At the start: 11 parts, among them J101 TT, J102 BT, U101 rp2040-zero

Commit message: 溜めすぎ　人間性0点
Parts:
- added J3: PSX, Connector_PinSocket_2.54mm:PinSocket_1x07_P2.54mm_Vertical, symbol Connector_Generic:Conn_01x07
- added JP1: PSX3V3, Connector_PinHeader_2.54mm:PinHeader_1x02_P2.54mm_Vertical, symbol Connector_Generic:Conn_01x02
- added R1, R2, R3, R4, R5, R6, R7: 1k, Resistor_THT:R_Axial_DIN0204_L3.6mm_D1.6mm_P5.08mm_Horizontal, symbol Device:R
- added R10, R11: 330, Resistor_SMD:R_0805_2012Metric_Pad1.20x1.40mm_HandSolder, symbol Device:R
- R8: renamed from R101; footprint Resistor_SMD:R_0805_2012Metric_Pad1.20x1.40mm_HandSolder -> Resistor_THT:R_Axial_DIN0204_L3.6mm_D1.6mm_P5.08mm_Horizontal; now not fitted
- R9: renamed from R102; footprint Resistor_SMD:R_0805_2012Metric_Pad1.20x1.40mm_HandSolder -> Resistor_THT:R_Axial_DIN0204_L3.6mm_D1.6mm_P5.08mm_Horizontal; now not fitted
- renumbered H101 to H1, H102 to H2, J101 to J1, J102 to J2, S101 to S1, S102 to S2, S103 to S3, S104 to S4, U101 to U1
Connections:
- net +3V3: now also JP1.2 (Pin_2), R1.2, R10.1, R11.1, R2.2, R3.2, R4.2, R5.2, R6.2, R7.2
- net GND: now also J3.7 (Pin_7)
- net KEY_1: now also R6.1
- net KEY_2: now also R7.1
- net KEY_3: now also R3.1
- net KEY_4: now also R4.1
- net KEY_5: now also R5.1
- net KEY_6: now also R2.1
- net KEY_7: now also R1.1
- net SCR_LEDA: now also R10.2
- net SCR_LEDB: now also R11.2
- net PSX_SCK: now reaches U1.17 (26)
- net PSX_SCK: now also J3.3 (Pin_3)
- net PSX_CMD: now reaches U1.18 (27)
- net PSX_CMD: now also J3.4 (Pin_4)
- net PSX_DAT: now reaches U1.19 (28)
- net PSX_DAT: now also J3.5 (Pin_5)
- net PSX_ACK: now reaches U1.20 (29)
- net PSX_ACK: now also J3.6 (Pin_6)
- net SCR_DOWN renamed PSX_ATT
- net PSX_ATT: now also J3.2 (Pin_2)
- net SCR_UP: no longer names the net of U1.15 (14)
- new net: J3.1 (Pin_1), JP1.1 (Pin_1)
- no-connect marks 9 -> 6
